Commit message: feat：增加dae模型文件

File: pix_planck_description/urdf/vehicle.xacro (robot description, xacro)
@@ -8,5 +8,5 @@
       <origin xyz="-0.25 0.0 0.1" rpy="0 0 ${pi/2.0}"/>
       <geometry>
-        <mesh filename="package://pix_planck_description/mesh/hooke.dae" scale="0.001 0.001 0.001"/>
+        <mesh filename="package://pix_planck_description/mesh/planck.dae" scale="0.001 0.001 0.001"/>
       </geometry>
     </visual>

Commit message: feat：Update vehicle.xacro

File: pix_planck_description/urdf/vehicle.xacro (robot description, xacro)
@@ -6,5 +6,5 @@
   <link name="base_link">
     <visual>
-      <origin xyz="-0.25 0.0 0.1" rpy="0 0 ${pi/2.0}"/>
+      <origin xyz="-0.25 0.0 0.1" rpy="0 0 0"/>
       <geometry>
         <mesh filename="package://pix_planck_description/mesh/planck.dae" scale="0.001 0.001 0.001"/>

Commit message: Update vehicle.xacro origin xyz

File: pix_planck_description/urdf/vehicle.xacro (robot description, xacro)
@@ -6,5 +6,5 @@
   <link name="base_link">
     <visual>
-      <origin xyz="-0.25 0.0 0.1" rpy="0 0 0"/>
+      <origin xyz="-0.5 0.0 0.0" rpy="0 0 0"/>
       <geometry>
         <mesh filename="package://pix_planck_description/mesh/planck.dae" scale="0.001 0.001 0.001"/>
